Commit message: Add end effector link

File: franka_description_gazebo/robots/panda.gazebo.xacro (robot description, xacro)
@@ -16,4 +16,11 @@
             </gazebo>
         </xacro:macro>
+        <xacro:macro name="end_effector_gazebo" params="link">
+            <gazebo reference="${link}">
+                <material>Gazebo/Red</material>
+                <mu1>0.2</mu1>
+                <mu2>0.2</mu2>
+            </gazebo>
+        </xacro:macro>
         <xacro:arm_gazebo link="${arm_id}_link0"/>
         <xacro:arm_gazebo link="${arm_id}_link1"/>
@@ -28,4 +35,5 @@
         <xacro:hand_gazebo link="${arm_id}_rightfinger"/>
         <xacro:hand_gazebo link="${arm_id}_leftfinger"/>
+        <xacro:end_effector_gazebo link="end_effector_link"/>
     </xacro:macro>
 </robot>

File: franka_description_gazebo/robots/panda_arm.xacro (robot description, xacro)
@@ -94,4 +94,26 @@
     <xacro:arm_joint name="${arm_id}_joint8" type="fixed" parent_link="${arm_id}_link7" child_link="${arm_id}_link8"
       rpy="0 0 0" xyz="0 0 0.107"/>
+    <!-- end effector joint -->
+    <joint name="end_effector_joint" type="fixed">
+      <origin xyz="0.0 0.0 0.2" rpy="0 0 0"/>
+      <parent link="${arm_id}_link7"/>
+      <child link="end_effector_link"/>
+    </joint>
+    <!-- end effector link -->
+    <link name="end_effector_link">
+      <visual>
+        <origin xyz="0 0 0" rpy="0 0 0"/>
+        <geometry>
+          <box size="0.01 0.01 0.01"/>
+        </geometry>
+       </visual>
+      <inertial>
+        <origin xyz="0 0 0"/>
+        <mass value="0.0"/>
+        <inertia ixx="0.001" ixy="0.0" ixz="0.0"
+                 iyy="0.001" iyz="0.0"
+                 izz="0.001"/>
+      </inertial>
+    </link>
   </xacro:macro>
 </robot>
